File: Hardware/pizza_clock.kicad_pcb (KiCad board)
At the start: 2 copper layers, 60 x 70 mm, 25 parts, among them J1 USB_C_Receptacle_PowerOnly_6P, J2 Conn_BAT, J3 Conn_USBASP, J4 Conn_rotary, Q1 PN2222A, U1 ATmega168-20A, U2 CA56-12CGKWA, U4 BQ24090DGQ

Commit message: update
Parts:
- removed D1: LED, LED_SMD:LED_0805_2012Metric
- removed J4: Conn_rotary, Connector_PinHeader_2.54mm:PinHeader_1x05_P2.54mm_Vertical
- added C4: 0.1uF, Capacitor_SMD:C_1206_3216Metric_Pad1.33x1.80mm_HandSolder, F.Cu at (78.3, 115.3)
- added C7: 0.1uF, Capacitor_SMD:C_1206_3216Metric_Pad1.33x1.80mm_HandSolder, F.Cu at (100.5, 109.8)
- added C8: 0.1uF, Capacitor_SMD:C_1206_3216Metric_Pad1.33x1.80mm_HandSolder, F.Cu at (95.7, 133.4)
- added C9: 0.1uF, Capacitor_SMD:C_1206_3216Metric_Pad1.33x1.80mm_HandSolder, F.Cu at (106.8, 133.5)
- added R11: 10K, Resistor_SMD:R_1206_3216Metric_Pad1.30x1.75mm_HandSolder, F.Cu at (85.7, 123.7)
- added R12: 220, Resistor_SMD:R_1206_3216Metric_Pad1.30x1.75mm_HandSolder, F.Cu at (78.2, 110.7)
- added R13: 10K, Resistor_SMD:R_1206_3216Metric_Pad1.30x1.75mm_HandSolder, F.Cu at (105.8, 109.8)
- added R14: 10K, Resistor_SMD:R_1206_3216Metric_Pad1.30x1.75mm_HandSolder, F.Cu at (95.6, 130.7)
- added R15: 10K, Resistor_SMD:R_1206_3216Metric_Pad1.30x1.75mm_HandSolder, F.Cu at (106.9, 130.8)
- added R16: 5K1, Resistor_SMD:R_1206_3216Metric_Pad1.30x1.75mm_HandSolder, F.Cu at (80.8, 139.6)
- added R17: 2K, Resistor_SMD:R_1206_3216Metric_Pad1.30x1.75mm_HandSolder, F.Cu at (126.7, 126.5)
- added SW1: RST, Button_Switch_SMD:SW_Tactile_SPST_NO_Straight_CK_PTS636Sx25SMTRLFS, F.Cu at (73.0, 112.3)
- added SW2: RotaryEncoder_Switch, Rotary_Encoder:RotaryEncoder_Alps_EC11E-Switch_Vertical_H20mm, F.Cu at (99.0, 127.8)
- D2: value LED -> RED
- D3: value LED -> BLUE
- R5: value 220 -> 5K1
- moved J3 64.9 mm to (124.5, 140.2), turned to 180 degrees
- moved J2 54.4 mm to (93.9, 146.2), turned to 0 degrees
- moved J1 54.1 mm to (82.5, 145.8), turned to 0 degrees
- moved R10 50.8 mm to (74.0, 128.2)
- moved D2 50.4 mm to (74.0, 132.8)
- moved U1 47.3 mm to (113.8, 140.6)
- moved C1 45.9 mm to (106.2, 140.0), turned to 90 degrees
- moved Q1 45.7 mm to (122.3, 126.3), turned to 90 degrees
- moved R9 45.1 mm to (71.0, 128.2), turned to -90 degrees
- moved R5 44.4 mm to (86.4, 139.3)
- moved R8 43.7 mm to (78.7, 134.2)
- moved D3 43.6 mm to (71.1, 132.8)
- moved C2 41.6 mm to (81.2, 132.9), turned to -90 degrees
- moved U2 36.7 mm to (93.5, 102.9)
- moved R7 36.2 mm to (75.4, 122.0), turned to 90 degrees
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Connections:
- net PB1 renamed B
- net PC4 renamed DPX
- J1 pad A5: unconnected-(J1-CC1-PadA5) -> Net-(J1-CC1)
- J1 pad B5: unconnected-(J1-CC2-PadB5) -> Net-(J1-CC2)
- J3 pad 1: GND -> RST
- J3 pad 2: RST -> GND
- J3 pad 3: MOSI -> SCK
- J3 pad 4: PB5 -> MOSI
- J3 pad 5: BAT+ -> MISO
- J3 pad 6: MISO -> BAT+
- Q1 pad 2: PC5 -> Net-(Q1-B)
- R1 pad 2: PC0 -> CA1
- R2 pad 2: PC1 -> CA2
- R3 pad 2: PC2 -> CA3
- R4 pad 2: PC3 -> CA4
- R5 pad 1: Net-(D1-A) -> Net-(J1-CC2)
- R5 pad 2: Net-(U1-PD2) -> GND
- U1 pad 1: unconnected-(U1-PD3-Pad1) -> CLK
- U1 pad 10: DT -> F
- U1 pad 11: CLK -> CA2
- U1 pad 12: PB0 -> CA3
- U1 pad 14: PB2 -> SW
- U1 pad 17: PB5 -> SCK
- U1 pad 18: unconnected-(U1-AVCC-Pad18) -> BAT+
- U1 pad 2: unconnected-(U1-PD4-Pad2) -> DT
- U1 pad 23: PC0 -> BUZZ
- U1 pad 24: PC1 -> CA4
- U1 pad 25: PC2 -> G
- U1 pad 26: PC3 -> C
- U1 pad 28: PC5 -> D
- U1 pad 32: Net-(U1-PD2) -> E
- U1 pad 8: unconnected-(U1-XTAL2/PB7-Pad8) -> CA1
- U1 pad 9: SW -> A
- U2 pad 1: MISO -> E
- U2 pad 10: PB5 -> F
- U2 pad 11: PB0 -> A
- U2 pad 2: MOSI -> D
- U2 pad 4: PB2 -> C
- U2 pad 5: PB6 -> G
Routing:
- net BAT+: track 125.0 -> 204.7 mm, vias 9 -> 2
- net A: track 0.00 -> 78.0 mm, vias 0 -> 1
- net F: track 0.00 -> 77.7 mm, vias 0 -> 1
- net CA3: track 0.00 -> 76.2 mm, vias 0 -> 2
- net CA2: track 0.00 -> 74.4 mm, vias 0 -> 2
- net CA1: track 0.00 -> 71.7 mm, vias 0 -> 2
- net MISO: track 71.0 -> 16.5 mm, vias 2 -> 1
- net B: track 27.6 -> 82.0 mm
- net PC3: track 53.3 -> 0.00 mm, vias 2 -> 0
- net RST: track 11.5 -> 64.7 mm, vias 0 -> 3
- net PB5: track 52.6 -> 0.00 mm, vias 4 -> 0
- net PB6: track 50.6 -> 0.00 mm, vias 1 -> 0
- net D: track 0.00 -> 49.2 mm
- net E: track 0.00 -> 47.4 mm
- net PB2: track 44.5 -> 0.00 mm, vias 2 -> 0
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Other:
- board text added: "Timer v3.0 Lucas Canete"
- board text removed: "C1"
- board text removed: "R2"
- board text removed: "Timer v2.0 Lucas Canete"
