File: Hardware/pizza_clock.kicad_sch (KiCad schematic)
At the start: 25 parts, among them J1 USB_C_Receptacle_PowerOnly_6P, J2 Conn_BAT, J3 Conn_USBASP, J4 Conn_rotary, Q1 PN2222A, U1 ATmega168-20A, U2 CA56-12CGKWA, U4 BQ24090DGQ

Commit message: update
Parts:
- removed D1: LED, LED_SMD:LED_0805_2012Metric, symbol Device:LED
- removed J4: Conn_rotary, Connector_PinHeader_2.54mm:PinHeader_1x05_P2.54mm_Vertical, symbol Connector:Conn_01x05_Pin
- added C4, C7, C8, C9: 0.1uF, Capacitor_SMD:C_1206_3216Metric_Pad1.33x1.80mm_HandSolder, symbol Device:C
- added R11, R13, R14, R15: 10K, Resistor_SMD:R_1206_3216Metric_Pad1.30x1.75mm_HandSolder, symbol Device:R
- added R12: 220, Resistor_SMD:R_1206_3216Metric_Pad1.30x1.75mm_HandSolder, symbol Device:R
- added R16: 5K1, Resistor_SMD:R_1206_3216Metric_Pad1.30x1.75mm_HandSolder, symbol Device:R
- added R17: 2K, Resistor_SMD:R_1206_3216Metric_Pad1.30x1.75mm_HandSolder, symbol Device:R
- added SW1: RST, Button_Switch_SMD:SW_Tactile_SPST_NO_Straight_CK_PTS636Sx25SMTRLFS, symbol Switch:SW_Push
- added SW2: RotaryEncoder_Switch, Rotary_Encoder:RotaryEncoder_Alps_EC11E-Switch_Vertical_H20mm, symbol Device:RotaryEncoder_Switch
- D2: value LED -> RED
- D3: value LED -> BLUE
- R5: value 220 -> 5K1
Connections:
- net CLK: now also U1.1 (PD3), C9.1, R15.1, SW2.B; no longer U1.11 (PD7)
- net DT: now also U1.2 (PD4), C8.1, R14.1, SW2.A; no longer U1.10 (PD6)
- net GND: now also J3.2 (Pin_2), R5.2, C4.2, C7.2, C8.2, C9.2, R16.2, SW1.1, SW2.C, SW2.S2; no longer J3.1 (Pin_1)
- net MISO: now also J3.5 (Pin_5); no longer J3.6 (Pin_6), U2.1 (e)
- net MOSI: now also J3.4 (Pin_4); no longer J3.3 (Pin_3), U2.2 (d)
- net PB6: no longer U2.5 (g)
- net RST: now also J3.1 (Pin_1), C4.1, R11.1, R12.2; no longer J3.2 (Pin_2)
- net SW: now also U1.14 (PB2), C7.1, R13.1, SW2.S1; no longer U1.9 (PD5)
- net VCC: now also J3.6 (Pin_6), U1.18 (AVCC), R11.2, R13.2, R14.2, R15.2; no longer J3.5 (Pin_5)
- net at R5.1: now also J1.B5 (CC2)
- net E: now reaches U1.32 (PD2)
- net E: now also U2.1 (e); no longer R5.2
- net CA1: now reaches U1.8 (XTAL2/PB7)
- net CA1: now also R1.2
- net at J1.A5 (CC1): now also R16.1
- net PB0 renamed A
- net A: now also U1.9 (PD5); no longer U1.12 (PB0)
- net PB1 renamed B
- net PB2 renamed C
- net C: now also U1.26 (PC3); no longer U1.14 (PB2)
- removed net PB5: J3.4 (Pin_4), U1.17 (PB5), U2.10 (f)
- net PC0 renamed BUZZ
- net BUZZ: now also R17.1; no longer R1.2
- net PC1 renamed CA2
- net CA2: now also U1.11 (PD7); no longer U1.24 (PC1)
- net PC2 renamed CA3
- net CA3: now also U1.12 (PB0); no longer U1.25 (PC2)
- net PC3 renamed CA4
- net CA4: now also U1.24 (PC1); no longer U1.26 (PC3)
- net PC4 renamed DPX
- net PC5: no longer names the net of Q1.2 (B)
- net PC5: now also R17.2; no longer U1.28 (PC5)
- new net: R12.1, SW1.2
- new net D: U1.28 (PC5), U2.2 (d)
- new net F: U1.10 (PD6), U2.10 (f)
- new net G: U1.25 (PC2), U2.5 (g)
- new net SCK: J3.3 (Pin_3), U1.17 (PB5)
- no-connect marks 9 -> 3
Other:
- note added: "AVCC to VCC so that port C has the same current as ports B and D"
- note added: "CHG LOW while charging (LED on while charging until threshold is reached) PG (Power Good) turns Low impedance when USB is connected PowerGood/USB present"
- note added: "Not enough pins for external clock"
- note added: "RESET"
- note added: "connect ISET2 to GND (LOW) to use current defined by R ISET connect ISET2 to VBUS (HIGH) to use current 500mA"
- note added: "not used"
- note added: "with 540 Ohm Resistor on ISET Iout = 1000mA"
- note removed: "540/Iout = 540 Iout = 1000mA"
- note removed: "CAMBIAR FOOTPRINT DE ATMEGA168"
- note removed: "CHG LOW while charging (LED on while charging until threshold is reached) PG (Power Good) turns Low impedance to ground when battery has reached good level (D3 turns on)"
- note removed: "Ideally for SMD compontents choose 1210 or 1206 because they are the biggest one. If not present 0805"
- note removed: "LED for signaling configuration purposes"
- note removed: "TO DO: -Calculate Value of resistors for the display (done)"
- moved on the sheet: BZ1, J3, Q1, R1, R2, R3, R4, U2
